Commit message: The calibrated mount goes into pose-mode IK too: robot.yaml arm_calibration, the planner URDF and arm_transform's fallbacks = inv(extrinsics T_ab2mb)
User: the corrected TF chain is for end-effector pose control as well as
map calibration. Until now only the locator chain (extrinsics.yaml) had
the 2026-09-21 calibration; pose-mode IK (transform_world_to_arm) still
used the design mount, so a tag located through the cameras and a
pose-mode target sent to the arm disagreed by ~25 mm / 1.4 deg on every
round trip. Now the same transform is in all three places that hold it:

- robot.yaml arm_calibration = inv(T_ab2mb) in the module's own
  parametrisation: offsets (-0.013008, -0.120318, 0.629002) m,
  mount_yaw 3.166578737 rad (181.43 deg), tilt_x/y 0.005926625 /
  0.013580283 rad. Exact reconstruction (R 1e-9). arm_transform.py's
  hardcoded fallbacks and docstring follow. arm_node restart required.
- planner URDF fr10v6_mobile_vision_0317_test.urdf mobile_to_base xyz
  (0.013008, 0.120318, 0.629002) rpy (0.005926625, 0.013580283,
  0.024986084) - the same transform seen from its 180-deg-yawed
  mobile_base. Existing rrt_final_path_* were planned with the design
  mount and now land ~45 mm from their assigned_workpoints_* twins until
  regenerated with this URDF.
- check_pose_vs_joint.py: asserts the three files agree; the planner-row
  convention tests run under the DESIGN block those rows were planned
  with, and the 45 mm discrepancy under the calibrated mount is asserted
  as expected rather than hidden (26). check_lift_compensation.py made
  tilt-aware - the lift is vertical in the WORLD, so with a 0.85 deg tilt
  the full stroke leaks 5 mm into arm x/y, which is right (11).
  check_scan_progress.py derived its IK-message numbers from the
  transform instead of the design-mount literals (49).

The applied roll/pitch are kept for consistency with the locator chain,
not as a mount measurement (+-1 deg, this parking's chassis attitude and
paper) - stated in robot.yaml, the URDF comment, CLAUDE.md and the
session record. Every pose-mode target moves ~35 mm at 1 m reach.

Co-Authored-By: Claude Opus 5 (1M context) <noreply@anthropic.com>

File: src/frcobot_ros/frcobot_description/urdf/fr10v6_mobile_vision_0317_test.urdf (robot description, URDF)
Before this commit: robot fr10v6_mobile, 11 links, 10 joints
Joints:
- joint mobile_to_base: origin xyz=0 0.1 0.652 rpy=0 0 0 -> xyz=0.013008 0.120318 0.629002 rpy=0.005926625 0.013580283 0.024986084

Commit message: vision tip APPLIED: (-1.8, -245.6, 209.6) mm in robot.yaml, set_tool_tcp.py and the planner URDF (measured 2026-09-21, verified on the robot); the RRT CSVs are stale for pose mode until re-exported
Co-Authored-By: Claude Opus 5 (1M context) <noreply@anthropic.com>

File: src/frcobot_ros/frcobot_description/urdf/fr10v6_mobile_vision_0317_test.urdf (robot description, URDF)
Before this commit: robot fr10v6_mobile, 11 links, 10 joints
Joints:
- joint vision_tip_joint: origin xyz=0 -0.25299 0.2252 rpy=0 0 0 -> xyz=-0.0018 -0.2456 0.2096 rpy=0 0 0

Commit message: Calibration set refit for the new hand_cam K: T_hc2ee re-solved from the 09-18 sweep frames (5.4 mm), arm joint zero offsets APPLIED to the locator chain (config/tf/arm_joint_offsets.yaml, FK(q+dq) via tf_chain.arm_flange_T; user's decision), T_ab2mb refit on the arm session with both (hold-out 12.7 -> 7.7 mm); URDF mobile_to_base follows; chain_calib.py --arm-offsets; check_joint_offsets 22
Co-Authored-By: Claude Opus 5 <noreply@anthropic.com>

File: src/frcobot_ros/frcobot_description/urdf/fr10v6_mobile_vision_0317_test.urdf (robot description, URDF)
Before this commit: robot fr10v6_mobile, 11 links, 10 joints
Joints:
- joint mobile_to_base: origin xyz=0.013008 0.120318 0.629002 rpy=0.005926625 0.013580283 0.024986084 -> xyz=0.006101 0.108596 0.642272 rpy=-0.007903911 -0.001687209 0.013726417

Commit message: T_ab2mb fitted PLANAR by rule (user): x, y, yaw only, roll = pitch = 0, tz = design — a sheet session's tilt is the chassis attitude at that parking and map calibration runs elsewhere; solver.fit_planar_T_ab2mb + chain_calib.py solve 'planar' row / T_ab2mb_planar in corrections.npz; applied t (-8.20, -106.13, -652.00) mm / yaw 179.196 deg, URDF mobile_to_base follows; checks 13 / 27 / 11 / 22 / 24 / 11 / 62 / 48
Co-Authored-By: Claude Opus 5 <noreply@anthropic.com>

File: src/frcobot_ros/frcobot_description/urdf/fr10v6_mobile_vision_0317_test.urdf (robot description, URDF)
Before this commit: robot fr10v6_mobile, 11 links, 10 joints
Joints:
- joint mobile_to_base: origin xyz=0.006101 0.108596 0.642272 rpy=-0.007903911 -0.001687209 0.013726417 -> xyz=0.006706 0.106230 0.652000 rpy=0.000000000 0.000000000 0.014030243

Commit message: T_ee2tip re-solved into the 2026-09-22 set (new hand-eye + checkerboard K: (-2.0, -245.2, 214.4) mm, the 09-21 pair reproduces the old value exactly); basler_tip --hand-intrinsics; applied to tf_chain, the URDF vision_tip_joint and the three tool-extent copies; calibration plans regenerated for the whole set (seeds 23 mm mean) — K -> T_hc2ee -> joint offsets -> T_ab2mb (planar) -> T_ee2tip are one set, tf_chain_tool check 13/13
Co-Authored-By: Claude Opus 5 <noreply@anthropic.com>

File: src/frcobot_ros/frcobot_description/urdf/fr10v6_mobile_vision_0317_test.urdf (robot description, URDF)
Before this commit: robot fr10v6_mobile, 11 links, 10 joints
Joints:
- joint vision_tip_joint: origin xyz=-0.0018 -0.2456 0.2096 rpy=0 0 0 -> xyz=-0.0020 -0.2452 0.2144 rpy=0 0 0

Commit message: 2026-09-28 working tree, all sessions: base stop poses per map tag (docs/robot_base_stop_poses.csv + tools/map_stop_poses.py), map.yaml 100-125 from the 16:14 / 21:33 sessions, T_ab2mb x,y shift, joint offsets on the command side (xy only), /robot_pose live stream + heading projection, arm reset_error, sheet_sweep + hand_cam intrinsics tools, the day's calibration / nav / tip-check records
- tools/map_stop_poses.py: where the mobile base CENTRE is (world x, y, yaw) when
  front_cam has aligned on a WORK tag and stopped on the FWD column — heading =
  zone axis + the tag's calibrated laying angle, base = tag - camera_offset along
  it; asserts from tf_chain.yaml that T_mb2fc @ T_tilted_to_level is exactly
  diag(1,-1,-1), so the physical tilt / yaw are already inside the level frame
  the align works in. Output docs/robot_base_stop_poses.csv, tags 100-150
  (--ids all for the rest). Reference data for the path generator.
- .gitignore: results/tip_check frames (80 Basler PNGs, 474 MB) excluded like
  results/scan_images; the tip-check yaml / csv records under log/ are versioned.
- Everything else: the uncommitted work of the other 2026-09-28 sessions as
  recorded in the CLAUDE.md Work Log entries of that day.

Co-Authored-By: Claude Fable 5.1 <noreply@anthropic.com>

File: src/frcobot_ros/frcobot_description/urdf/fr10v6_mobile_vision_0317_test.urdf (robot description, URDF)
Before this commit: robot fr10v6_mobile, 11 links, 10 joints
Joints:
- joint mobile_to_base: origin xyz=0.006706 0.106230 0.652000 rpy=0.000000000 0.000000000 0.014030243 -> xyz=0.007804 0.099245 0.652000 rpy=0.000000000 0.000000000 0.014030243

Commit message: Vision tip = DESIGN of the new case mesh; config stage 1: one place for the tip, kind: markers, docs/FRAMES_kr.md
- visionsystem_final.stl (CAD export 2026-10-11) replaces vision_system_total_DF_1031.stl in the planner URDF's `vision` link; the export is not in the flange frame, so the link origin rpy(-90, 0, 180) deg xyz(-117.6, -7.15, -20.6) mm puts its 63x80 mm flange plate on z=0 (matched to the old mesh's identical plate face: 144 tris, same area).
- tf_chain.yaml T_ee2tip set (tf_chain_tool.py set) to the DESIGN tip (0.12, -251.96, 222.0) mm: the new mesh's lens axis (common centre of the rings at z 64 / 126 / 192-196, tilt 0.02 deg vs flange z), 16 mm below the case end (z 206.0); the 2026-09-22 measurement (-2.0, -245.2, 214.4) stays as the measured_2026_09_22 sub-block. NOT measured on the robot - re-measure with the new case; arm_node restart and a planner re-export of task/csv are still open.
- Planner URDF vision_tip_joint follows (check: 13 ok). The tip copies in generate_calibration_artifacts.py (TOOL_OFFSET_MM) and handeye_sweep.SweepCfg.tool_points_mm (+ the handeye_calib.yaml line) now read tf_chain.tip_offset_mm().
- tf_chain.yaml: `kind:` per block (calibrated / generated / design); arm_joint_offsets.yaml paths -> ${MM_WS}.
- docs/FRAMES_kr.md: frames, conventions, where every number lives, recalibration recipes. CLAUDE.md Work Log entry.

Verified offline: tf_chain_tool.py check 0 failed; check_joint_offsets 22, check_ground_plane 15, check_front_cam_pose_calib 28, check_lift_compensation 9, check_handeye_sweep 74. Not run on the robot.

Co-Authored-By: Claude Fable 5.1 <noreply@anthropic.com>

File: src/frcobot_ros/frcobot_description/urdf/fr10v6_mobile_vision_0317_test.urdf (robot description, URDF)
Before this commit: robot fr10v6_mobile, 11 links, 10 joints
Links:
- link vision: geometry collision mesh filename=../../meshes/fr10v6_meshes_0126/fr10v6/visual/visionsystem_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 scale=0.001 0.001 0.001; visual mesh filename=../../meshes/fr10v6_meshes_0126/fr10v6/visual/visionsystem_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 scale=0.001 0.001 0.001
Joints:
- joint vision_tip_joint: origin xyz=-0.0020 -0.2452 0.2144 rpy=0 0 0 -> xyz=0.00012 -0.25196 0.2220 rpy=0 0 0

Commit message: Config stage 4: tf_chain_tool.py urdf --apply writes the planner URDF's mobile_to_base / vision_tip_joint lines in place
- tf_chain.py: urdf_joint_lines(), read_urdf_joint(), write_urdf_joints() — replaces exactly the two <origin .../> lines (every other byte stays), numeric change test (1e-6 m / 1e-7 rad: formatting-only differences are left alone), refuses a missing joint or vision_fixed off 0, re-reads and verifies after writing; planner_urdf_path().
- tf_chain_tool.py: `urdf` shows was/now, `urdf --apply` writes; top-level --urdf PATH for check / urdf / show.
- URDF: vision_tip_joint z "0.2220" -> "0.22200" (textual only; values identical, check 0 failed).
- check_tf_chain_yaml.py: +12 checks on a copy of the URDF (dry no-op, apply after a tip change touches one line, check --urdf passes, idempotent, refusals, real file untouched) — 52 total.
- docs/FRAMES_kr.md recipes, CLAUDE.md Work Log.

Verified offline: check 0 failed, check_tf_chain_yaml 52, check_tf_chain_publisher 27, stage-1 checks unchanged. Nothing runs on the robot.

Co-Authored-By: Claude Fable 5.1 <noreply@anthropic.com>

File: src/frcobot_ros/frcobot_description/urdf/fr10v6_mobile_vision_0317_test.urdf (robot description, URDF)
Before this commit: robot fr10v6_mobile, 11 links, 10 joints
Joints:
- joint vision_tip_joint: origin xyz=0.00012 -0.25196 0.2220 rpy=0 0 0 -> xyz=0.00012 -0.25196 0.22200 rpy=0 0 0
