Commit message: Design tip z 222.0 -> 223.0 mm: the case end-to-tip distance is 17 mm, not 16 (user, 2026-10-19). tf_chain.yaml T_ee2tip (0.12, -251.96, 223.0) via set --kind design, design sub-block + note, urdf --apply on fr10v6_mobile_visionsystem_final.urdf, FRAMES_kr / CLAUDE.md. check 0 failed, check_tf_chain_yaml 52, check_tf_chain_publisher 27.
Co-Authored-By: Claude Fable 5.1 <noreply@anthropic.com>

File: src/frcobot_ros/frcobot_description/urdf/fr10v6_mobile_visionsystem_final.urdf (robot description, URDF)
Before this commit: robot fr10v6_mobile, 11 links, 10 joints
Joints:
- joint vision_tip_joint: origin xyz=0.00012 -0.25196 0.22200 rpy=0 0 0 -> xyz=0.00012 -0.25196 0.22300 rpy=0 0 0
